File: Lid/FLAP_Panel.brd (EAGLE design)
At the start: 7 parts

Commit message: Lid and flap file cleanup
Parts:
- removed FRAME1: FRAME-LETTER, SparkFun-Aesthetics:CREATIVE_COMMONS
- added E$10, E$11, E$12, E$13, E$15, E$16, E$17, E$18, E$19, E$20, E$21, E$22, E$23, E$24, E$25, E$26, E$27, E$29, E$30, E$31, E$32, E$33, E$34, E$35, E$36, E$37, E$38, E$39, E$4, E$40, E$41, E$6, E$9: (no value), lid:FLAP_1_8TH
- E$1: device lid:CAN_DIA -> lid:FLAP_1_8TH
- E$2: device snake:LID -> lid:FLAP_1_8TH
- E$3, E$7, E$8: device lid:LID_THICKNESS_060 -> lid:FLAP_1_8TH
- moved E$7 608.4 mm to (534.7, 274.3), turned to 270 degrees
- moved E$5 462.3 mm to (372.1, 274.3), turned to 270 degrees
- moved E$2 356.1 mm to (128.3, 274.3), turned to 270 degrees
- moved E$3 344.2 mm to (209.6, 274.3), turned to 270 degrees
- moved E$8 282.7 mm to (87.6, 232.4), turned to 270 degrees
- moved E$1 278.3 mm to (47.0, 274.3), turned to 270 degrees
Other:
- board text removed: "OLD radius: 1.015 NEW: 1.018 NEWEST: 1.021"
- board text removed: "Pete Lewis"
